Commit message: 5-dim functionality

File: robots/4DOFBoxRoboticArm.urdf (robot description, URDF)
Before this commit: robot simple_4dofbox, 5 links, 4 joints
Joints:
- joint joint1: limit lower=-3 upper=3 effort=5 velocity=1 -> lower=-1.57 upper=1.57 effort=5 velocity=1; origin xyz=0 0 0.15 rpy=0 0 0 -> xyz=0 0 0.1 rpy=0 0 0
- joint joint2: limit lower=-3 upper=3 effort=5 velocity=1 -> lower=0.0 upper=1.57 effort=5 velocity=1
- joint joint3: limit lower=-3 upper=3 effort=5 velocity=1 -> lower=-1.57 upper=1.57 effort=5 velocity=1
- joint joint4: limit lower=-3 upper=3 effort=5 velocity=1 -> lower=-1.57 upper= effort=1.57 velocity=1

File: robots/PackBot.urdf (robot description, URDF)
Before this commit: robot SCARA, 6 links, 5 joints
Links:
- removed link dummy_link
- removed link ee
- added link dummy, mass 1.0; collision box size=0.1 0.1 0.4; visual box size=0.0 0.0 0.0
- added link link4, mass 0.5; collision box size=0.1 0.1 0.3; visual box size=0.3 0.3 0.3
- link base_link: geometry collision cylinder length=0.1 radius=0.05; visual cylinder length=0.6 radius=0.15
- link link1: mass 0.8 -> 1.0; geometry collision box size=0.1 0.1 0.4; visual box size=0.2 0.2 1.0
- link link2: mass 0.5 -> 0.8; geometry collision box size=0.1 0.1 0.4; visual box size=0.2 0.2 1.25
- link link3: geometry collision box size=0.1 0.1 0.4; visual box size=0.2 0.2 1.25
Joints:
- joint joint1: child link1 -> dummy; limit lower=-1.8326 upper=1.8326 effort=5 velocity=1 -> lower=-1.57 upper=1.57 effort=5 velocity=1; origin xyz=0 0 1.05 rpy=0 0 0.7 -> xyz=0 0 0.1 rpy=0 0 0
- joint joint2: axis 0 0 1 -> 0 1 0; child link2 -> link1; limit lower=-2.7489 upper=2.7489 effort=5 velocity=1 -> lower=-1.27 upper=1.27 effort=5 velocity=1; origin xyz=0 0.4 0.1 rpy=0 0 0 -> xyz=0 0 0.3 rpy=0 0 0; parent link1 -> dummy
- joint joint3: axis 0 0 1 -> 0 1 0; child dummy_link -> link2; limit lower=-3 upper=3 effort=5 velocity=1 -> lower=-2.57 upper=2.57 effort=5 velocity=1; origin xyz=0 0.45 -0.45 rpy=0 0 0 -> xyz=0 0 1.0 rpy=0 0 0; parent link2 -> link1
- joint joint4: axis 0 0 1 -> 0 1 0; limit lower=-0.06 upper=0.1 effort=5 velocity=1 -> lower=-2.57 upper=2.57 effort=5 velocity=1; origin xyz=0 0 0.05 rpy=0 0 0 -> xyz=0 0 1.2 rpy=0 0 0; parent dummy_link -> link2; type prismatic -> revolute
- joint joint5: axis 0 0 1 -> 0 1 0; child ee -> link4; limit lower=-3 upper=3 effort=5 velocity=1 -> lower=-0.1 upper=0.1 effort=1.57 velocity=1; origin xyz=0 0 -0.45 rpy=0 0 0 -> xyz=0 0 1.2 rpy=0 0 0; type fixed -> revolute

File: robots/PackBotdummy.urdf (robot description, URDF)
Before this commit: robot SCARA, 6 links, 5 joints
Links:
- removed link dummy_link
- removed link ee
- added link dummy, mass 1.0; collision box size=0.1 0.1 0.4; visual box size=0.0 0.0 0.0
- added link link4, mass 0.5; collision box size=0.1 0.1 0.3; visual box size=0.3 0.3 0.3
- link base_link: geometry collision cylinder length=0.1 radius=0.05; visual cylinder length=0.6 radius=0.15
- link link1: mass 0.8 -> 1.0; geometry collision box size=0.1 0.1 0.4; visual box size=0.2 0.2 1.0
- link link2: mass 0.5 -> 0.8; geometry collision box size=0.1 0.1 0.4; visual box size=0.2 0.2 1.25
- link link3: geometry collision box size=0.1 0.1 0.4; visual box size=0.2 0.2 1.25
Joints:
- joint joint1: child link1 -> dummy; limit lower=-1.8326 upper=1.8326 effort=5 velocity=1 -> lower=-3 upper=3 effort=5 velocity=1; origin xyz=0 0 1.05 rpy=0 0 0.7 -> xyz=0 0 0.1 rpy=0 0 0
- joint joint2: axis 0 0 1 -> 0 1 0; child link2 -> link1; limit lower=-2.7489 upper=2.7489 effort=5 velocity=1 -> lower=-3 upper=3 effort=5 velocity=1; origin xyz=0 0.4 0.1 rpy=0 0 0 -> xyz=0 0 0.3 rpy=0 0 0; parent link1 -> dummy
- joint joint3: axis 0 0 1 -> 0 1 0; child dummy_link -> link2; origin xyz=0 0.45 -0.45 rpy=0 0 0 -> xyz=0 0 1.0 rpy=0 0 0; parent link2 -> link1
- joint joint4: axis 0 0 1 -> 0 1 0; limit lower=-0.06 upper=0.1 effort=5 velocity=1 -> lower=-3 upper=3 effort=5 velocity=1; origin xyz=0 0 0.05 rpy=0 0 0 -> xyz=0 0 1.2 rpy=0 0 0; parent dummy_link -> link2; type prismatic -> revolute
- joint joint5: axis 0 0 1 -> 0 1 0; child ee -> link4; limit lower=-3 upper=3 effort=5 velocity=1 -> lower=-1 upper=1 effort=5 velocity=1; origin xyz=0 0 -0.45 rpy=0 0 0 -> xyz=0 0 1.2 rpy=0 0 0; type fixed -> revolute

File: robots/ShoulderJointdummy.urdf (robot description, URDF)
Before this commit: robot SCARA, 6 links, 5 joints
Links:
- removed link dummy_link
- removed link ee
- added link link4, mass 0.5; collision box size=0.1 0.1 0.3; visual box size=0.1 0.1 0.5
- link base_link: geometry collision cylinder length=0.1 radius=0.05; visual sphere radius=0.1
- link link1: mass 0.8 -> 1.0; geometry collision box size=0.1 0.1 0.5; visual box size=0.0 0.0 0.0
- link link2: mass 0.5 -> 0.8; geometry collision box size=0.1 0.1 0.5; visual box size=0.0 0.0 0.0
- link link3: geometry collision box size=0.1 0.1 0.3; visual box size=0.1 0.1 0.7
Joints:
- removed joint joint5
- joint joint1: limit lower=-1.8326 upper=1.8326 effort=5 velocity=1 -> lower=0.0 upper=1.57 effort=5 velocity=1; origin xyz=0 0 1.05 rpy=0 0 0.7 -> xyz=0 0 0.0 rpy=0 0 0
- joint joint2: axis 0 0 1 -> 0 1 0; limit lower=-2.7489 upper=2.7489 effort=5 velocity=1 -> lower=0.0 upper=1.57 effort=5 velocity=1; origin xyz=0 0.4 0.1 rpy=0 0 0 -> xyz=0 0 0.0 rpy=0 0 0
- joint joint3: axis 0 0 1 -> 1 0 0; child dummy_link -> link3; limit lower=-3 upper=3 effort=5 velocity=1 -> lower=0.0 upper=1.57 effort=5 velocity=1; origin xyz=0 0.45 -0.45 rpy=0 0 0 -> xyz=0 0 0.0 rpy=0 0 0
- joint joint4: axis 0 0 1 -> 0 1 0; child link3 -> link4; limit lower=-0.06 upper=0.1 effort=5 velocity=1 -> lower=-1.57 upper=1.57 effort=5 velocity=1; origin xyz=0 0 0.05 rpy=0 0 0 -> xyz=0 0 0.7 rpy=0 0 0; parent dummy_link -> link3; type prismatic -> revolute
