Commit message: New scenes and fixed coxeter

File: robots/4DOFBoxRoboticArm.urdf (robot description, URDF)
Before this commit: robot simple_4dofbox, 5 links, 4 joints
Links:
- link base_link: mass 1.0 -> None; geometry collision cylinder length=0.1 radius=0.1; visual cylinder length=0.1 radius=0.1
- link link1: mass 1.0 -> None; geometry collision box size=0.1 0.1 0.5; visual box size=0.1 0.1 0.5
- link link2: geometry collision box size=0.1 0.1 0.5; visual box size=0.1 0.1 0.5
- link link3: mass 0.5 -> None; geometry collision box size=0.1 0.1 0.3; visual box size=0.1 0.1 0.3
- link link4: mass 0.5 -> None; geometry collision box size=0.1 0.1 0.3; visual box size=0.1 0.1 0.3
Joints:
- joint joint4: limit lower=-1.57 upper= effort=1.57 velocity=1 -> lower=-1.57 upper=1.57 effort=1.57 velocity=1

File: robots/6DOF.urdf (robot description, URDF)
Before this commit: robot simple_5dof, 6 links, 5 joints
Links:
- added link link5, mass 0.5; collision box size=0.1 0.1 0.3; visual box size=0.15 0.15 0.45
- link base_link: mass None -> 1.0; geometry collision cylinder length=0.1 radius=0.05; visual cylinder length=0.2 radius=0.1
- link dummy_link_1: mass None -> 1.0
- link link1: mass None -> 1.0; geometry collision box size=0.1 0.1 0.5; visual box size=0.15 0.15 0.75
- link link2: mass None -> 0.8; geometry collision box size=0.1 0.1 0.5; visual box size=0.15 0.15 0.5
- link link3: mass None -> 0.5; geometry collision box size=0.1 0.1 0.3; visual box size=0.15 0.45 0.15
- link link4: mass None -> 0.5; geometry collision box size=0.1 0.1 0.3; visual box size=0.15 0.15 0.45
Joints:
- added joint joint6: type revolute, parent link4, child link5, origin xyz=0 0.0 0.45 rpy=0 0 0, axis 0 1 0, limit lower=-0.2 upper=0.2 effort=5 velocity=1

File: robots/PackBotdummy.urdf (robot description, URDF)
Before this commit: robot simple_4dofbox, 6 links, 5 joints
Links:
- link base_link: mass 1.0 -> None; geometry collision cylinder length=0.6 radius=0.15; visual cylinder length=0.6 radius=0.15
- link dummy: mass 1.0 -> None; geometry collision box size=0.0 0.0 0.0; visual box size=0.0 0.0 0.0
- link link1: mass 1.0 -> None; geometry collision box size=0.2 0.2 1.0; visual box size=0.2 0.2 1.0
- link link2: mass 0.8 -> None; geometry collision box size=0.2 0.2 1.25; visual box size=0.2 0.2 1.25
- link link3: mass 0.5 -> None; geometry collision box size=0.2 0.2 1.25; visual box size=0.2 0.2 1.25
- link link4: mass 0.5 -> None; geometry collision box size=0.3 0.3 0.3; visual box size=0.3 0.3 0.3

File: robots/ShoulderJointdummy.urdf (robot description, URDF)
Before this commit: robot ShoulderJoint, 5 links, 4 joints
Links:
- link base_link: mass 1.0 -> None; geometry visual sphere radius=0.0
- link link1: mass 1.0 -> None; geometry collision box size=0.1 0.1 0.5; visual box size=0.0 0.0 0.0
- link link2: mass 0.8 -> None; geometry collision box size=0.0 0.0 0.0; visual box size=0.0 0.0 0.0
- link link3: mass 0.5 -> None; geometry collision box size=0.1 0.1 0.7; visual box size=0.1 0.1 0.7
- link link4: mass 0.5 -> None; geometry collision box size=0.1 0.1 0.5; visual box size=0.1 0.1 0.5
Joints:
- joint joint2: limit lower=0.0 upper=1.57 effort=5 velocity=1 -> lower=0 upper=1.57 effort=5 velocity=1
- joint joint3: limit lower=0.0 upper=1.57 effort=5 velocity=1 -> lower=-0.785 upper=0.785 effort=5 velocity=1
- joint joint4: limit lower=-1.57 upper=1.57 effort=5 velocity=1 -> lower=0 upper=1.57 effort=5 velocity=1
